Commit message: add controller

File: src/hakuroukun/hakuroukun_description/urdf/hakuroukun.urdf.xacro (robot description, xacro)
@@ -1,103 +1,113 @@
 <?xml version="1.0"?>
-<robot xmlns:xacro="http://ros.org/wiki/xacro" name="hakuroukun">
-  <!-- Constant -->
-  <!-- <xacro:property name="bottom_plate_to_wheel_plate" value="0.0625"/>
-  <xacro:property name="distance_two_wheel_plate" value="0.46"/>
-  <xacro:property name="wheel_plate_length" value="0.265"/>
-  <xacro:property name="wheel_radius" value="0.115"/>
-  <xacro:property name="wheel_length" value="0.09"/>
-  <xacro:property name="base_width" value="0.125"/>
-  <xacro:property name="base_length" value="0.7"/>
-  <xacro:property name="device_frame_to_base_front" value="0.14"/>
-  <xacro:property name="basket_length" value="0.645"/> -->
-  <xacro:property name="backwheel_axis_length" value="0.8" />
-  <xacro:property name="backwheel_axis_to_frontwheel_axis" value="1" />
-  <xacro:property name="wheel_radius" value="0.125" />
-  <xacro:property name="base_link_to_trunk_z" value="0.35" />
-  <xacro:property name="trunk_to_front_y" value="0.35" />
-  <xacro:property name="trunk_to_saddle_z" value="0.35" />
-  <!-- Material color -->
-  <!-- <material name="light steel blue">
-    <color rgba="${176/255} ${196/255} ${222/255} 1"/>
-  </material>
-  <material name="slate gray">
-    <color rgba="${112/255} ${128/255} ${144/255} 1"/>
-  </material>
-  <material name="cadet blue">
-    <color rgba="${95/255} ${158/255} ${160/255} 1"/>
-  </material> -->
-  <!-- Extras -->
-  <xacro:arg name="robot_namespace" default="$(optenv ROBOT_NAMESPACE /)" />
-  <!-- Included URDF/XACRO Files -->
-  <xacro:include filename="$(find hakuroukun_description)/urdf/robot_part/hakuroukun_base_link.urdf.xacro" />
-  <xacro:include filename="$(find hakuroukun_description)/urdf/robot_part/hakuroukun_right_backwheel.urdf.xacro" />
-  <xacro:include filename="$(find hakuroukun_description)/urdf/robot_part/hakuroukun_left_backwheel.urdf.xacro" />
-  <xacro:include filename="$(find hakuroukun_description)/urdf/robot_part/hakuroukun_frontwheel.urdf.xacro" />
-  <!-- <xacro:property name="caster_wheel_yaml" value="$(find hakuroukun_description)/config/diffbot/caster_wheel.yaml" />
-  <xacro:property name="caster_wheel_props" value="${xacro.load_yaml(caster_wheel_yaml)}"/> -->
-  <!-- Base_link macros -->
-  <xacro:hakuroukun_base_link/>
-  <!-- Base footprint is on the ground under the robot -->
-  <link name="base_footprint"/>
-  <joint name="base_footprint_joint" type="fixed">
-    <origin xyz="0 0 -wheel_radius" rpy="0 0 0" />
-    <parent link="base_footprint" />
-    <child link="base_link" />
-  </joint>
-  <!-- Left BackWheel macros -->
-  <xacro:hakuroukun_left_backwheel wheel_prefix="left_backwheel">
-    <origin xyz="-${backwheel_axis_length/2} 0 0" rpy="0 0 0" />
-  </xacro:hakuroukun_left_backwheel>
-  <!-- Right BackWheel macros -->
-  <xacro:hakuroukun_right_backwheel wheel_prefix="right_backwheel">
-    <origin xyz="${backwheel_axis_length/2} 0 0" rpy="0 0 0" />
-  </xacro:hakuroukun_right_backwheel>
-  <!-- FrontWheel macros -->
-  <xacro:hakuroukun_frontwheel wheel_prefix="front_wheel">
-    <origin xyz="0 ${backwheel_axis_to_frontwheel_axis} 0" rpy="0 0 0" />
-  </xacro:hakuroukun_frontwheel>
-  <!-- Back Caster Wheel -->
-  <!-- <xacro:caster_wheel prefix="left" reflect="-1" dx="${distance_two_wheel_plate/2}" dy="${wheel_plate_length/2-0.02}"
-    wheel_props="${caster_wheel_props}">
-  </xacro:caster_wheel>
-  <xacro:caster_wheel prefix="right" reflect="-1" dx="${distance_two_wheel_plate/2}" dy="-${wheel_plate_length/2-0.02}"
-    wheel_props="${caster_wheel_props}">
-  </xacro:caster_wheel> -->
-  <!-- Gazebo plugin for ROS Control -->
+<robot name="bicycle_bot" xmlns:xacro="http://wiki.ros.org/xacro">
+  <!-- Include xacro for inertials, materials and wheels -->
+  <xacro:include filename="$(find hakuroukun_description)/urdf/robot_part/wheel.xacro"/>
+  <xacro:property name="robot_namespace" value="hakuroukun"/>
+  <!-- Gazebo plugins -->
   <gazebo>
+    <!-- Load ros_control plugin -->
     <plugin name="gazebo_ros_control" filename="libgazebo_ros_control.so">
-      <robotNamespace>$(arg robot_namespace)</robotNamespace>
+      <robotNamespace>${robot_namespace}</robotNamespace>
+      <robotSimType>gazebo_ros_control/DefaultRobotHWSim</robotSimType>
+      <legacyModeNS>false</legacyModeNS>
+    </plugin>
+    <!-- Load gazebo_ros plugin. Publish passive (non-actuated) joints from Gazebo -->
+    <plugin name="gazebo_ros_joint_state_publisher" filename="libgazebo_ros_joint_state_publisher.so">
+        <robotNamespace>${robot_namespace}</robotNamespace>
+        <jointName>
+            front_wheel_joint
+        </jointName>
+        <updateRate>50</updateRate>
+        <alwaysOn>true</alwaysOn>
     </plugin>
   </gazebo>
-  <!-- Gazebo plugin for IMU -->
-  <gazebo>
-    <plugin name="imu_controller" filename="libhector_gazebo_ros_imu.so">
-      <robotNamespace>$(arg robot_namespace)</robotNamespace>
-      <updateRate>50.0</updateRate>
-      <bodyName>base_link</bodyName>
-      <topicName>imu/data</topicName>
-      <accelDrift>0.005 0.005 0.005</accelDrift>
-      <accelGaussianNoise>0.005 0.005 0.005</accelGaussianNoise>
-      <rateDrift>0.005 0.005 0.005 </rateDrift>
-      <rateGaussianNoise>0.005 0.005 0.005 </rateGaussianNoise>
-      <headingDrift>0.005</headingDrift>
-      <headingGaussianNoise>0.005</headingGaussianNoise>
-    </plugin>
-  </gazebo>
-  <!-- Gazebo plugin for GNSS -->
-  <gazebo>
-    <plugin name="gps_controller" filename="libhector_gazebo_ros_gps.so">
-      <robotNamespace>$(arg robot_namespace)</robotNamespace>
-      <updateRate>40</updateRate>
-      <bodyName>base_link</bodyName>
-      <frameId>gps_link</frameId>
-      <topicName>navsat/fix</topicName>
-      <velocityTopicName>navsat/vel</velocityTopicName>
-      <referenceLatitude>$(arg origin_lat)</referenceLatitude>
-      <referenceLongitude>$(arg origin_lon)</referenceLongitude>
-      <referenceHeading>180</referenceHeading>
-      <referenceAltitude>0</referenceAltitude>
-      <drift>0.0001 0.0001 0.0001</drift>
-    </plugin>
+  <!-- Math constants -->
+  <xacro:property name="deg_to_rad" value="0.01745329251994329577"/>
+  <!-- Robot base dimensions -->
+  <xacro:property name="base_length" value="1.35" />
+  <xacro:property name="base_width" value="0.8" />
+  <xacro:property name="base_height" value="1.1" />
+  <xacro:property name="base_mass" value="30" />
+  <!-- Wheel link dimensions -->
+  <xacro:property name="wheel_radius" value="0.125" />
+  <xacro:property name="wheel_thickness" value="0.1" />
+  <xacro:property name="wheel_mass" value="2" />
+  <!-- Steering link dimensions -->
+  <xacro:property name="steer_radius" value="0.05" />
+  <xacro:property name="steer_thickness" value="0.02" />
+  <xacro:property name="steer_mass" value="0.1" />
+  <!-- Axle positions -->
+  <xacro:property name="axle_offset" value="0.05" />
+  <xacro:property name="steer_offset" value="0.02" />
+  <xacro:property name="b2f_axis_distance" value="1.1"/>
+  <xacro:property name="b_axis_length" value="0.8"/>
+  <!-- Base link -->
+  <link name="base_link">
+    <visual>
+      <origin xyz="0 0 0" rpy="0 0 0"/>
+      <geometry>
+          <mesh filename="package://hakuroukun_description/meshes/hakuroukun_base_link.stl" scale="0.001 0.001 0.001" />
+      </geometry>
+      <material name="grey"/>
+    </visual>
+    <collision>
+      <origin xyz="0 0 0" rpy="0 0 0"/>
+      <geometry>
+          <mesh filename="package://hakuroukun_description/meshes/hakuroukun_base_link.stl" scale="0.001 0.001 0.001" />
+      </geometry>
+    </collision>
+    <xacro:solid_cuboid_inertial
+        rpy="0 0 0" xyz="0 0 0"
+        mass="${base_mass}"
+        x="${base_length}" y="${base_width}" z="${base_height}" />
+  </link>
+  <!-- Front steer and rear wheel joints required for ackermann_steering_controller -->
+  <xacro:front_steer
+    name="front"
+    parent="base"
+    steer_radius="${steer_radius}"
+    steer_thickness="${steer_thickness}"
+    steer_mass="${steer_mass}"
+    base_length="${base_length}"
+    base_width="${base_width}"
+    axle_offset="${axle_offset}"
+    steer_height="${wheel_radius+steer_offset}">
+  </xacro:front_steer>
+  <xacro:front_wheel
+    name="front"
+    parent="front_steer"
+    wheel_radius="${wheel_radius}"
+    wheel_thickness="${wheel_thickness}"
+    wheel_mass="${wheel_mass}">
+    <origin xyz="0 0 ${-wheel_radius-steer_offset}" rpy="0 0 ${90 * deg_to_rad}"/>
+  </xacro:front_wheel>
+  <!-- REAR WHEEL-->
+  <xacro:rear_wheel
+    name="rear"
+    parent="base"
+    wheel_radius="${wheel_radius}"
+    wheel_thickness="${wheel_thickness}"
+    wheel_mass="${wheel_mass}">
+    <origin xyz="0 0 0" rpy="0 0 0"/>
+  </xacro:rear_wheel>
+  <xacro:rear_wheel_lr
+    name="rear_right"
+    parent="base"
+    wheel_radius="${wheel_radius}"
+    wheel_thickness="${wheel_thickness}"
+    wheel_mass="${wheel_mass}">
+    <origin xyz="0 ${-b_axis_length/2} 0" rpy="0 0 0"/>
+  </xacro:rear_wheel_lr>
+  <xacro:rear_wheel_lr
+    name="rear_left"
+    parent="base"
+    wheel_radius="${wheel_radius}"
+    wheel_thickness="${wheel_thickness}"
+    wheel_mass="${wheel_mass}">
+    <origin xyz="0 ${b_axis_length/2} 0" rpy="0 0 0"/>
+  </xacro:rear_wheel_lr>
+  <!-- Colour -->
+  <gazebo reference="base_link">
+    <material>Gazebo/Green</material>
   </gazebo>
 </robot>
