Commit message: :rabbit: Build Hakuroukun Hardware Gazebo

File: src/hakuroukun/hakuroukun_description/urdf/backup/hakuroukun.urdf copy.xacro (robot description, xacro)
@@ -1,20 +1,23 @@
 <?xml version="1.0"?>
-<!--
-    For this model:
-    wheel_separation_h = 1.1
-    wheel_separation_w = 0.8
--->
-<robot name="hakuroukun" xmlns:xacro="http://wiki.ros.org/xacro">
+<robot name="bicycle_bot" xmlns:xacro="http://wiki.ros.org/xacro">
   <!-- Include xacro for inertials, materials and wheels -->
   <xacro:include filename="$(find hakuroukun_description)/urdf/robot_part/hakuroukun_wheel.xacro"/>
-  <xacro:property name="robot_namespace" value="/hakuroukun"/>
+  <xacro:property name="robot_namespace" value="hakuroukun"/>
   <!-- Gazebo plugins -->
   <gazebo>
-    <!-- Load ros_control plugin using the steer_bot_hardware_gazebo
-    implementation of the hardware_interface::RobotHW -->
+    <!-- Load ros_control plugin -->
     <plugin name="gazebo_ros_control" filename="libgazebo_ros_control.so">
       <robotNamespace>${robot_namespace}</robotNamespace>
-      <robotSimType>hakuroukun_hardware_gazebo/HakuroukunHardwareGazebo</robotSimType>
+      <robotSimType>gazebo_ros_control/DefaultRobotHWSim</robotSimType>
       <legacyModeNS>false</legacyModeNS>
+    </plugin>
+    <!-- Load gazebo_ros plugin. Publish passive (non-actuated) joints from Gazebo -->
+    <plugin name="gazebo_ros_joint_state_publisher" filename="libgazebo_ros_joint_state_publisher.so">
+        <robotNamespace>${robot_namespace}</robotNamespace>
+        <jointName>
+            front_wheel_joint
+        </jointName>
+        <updateRate>50</updateRate>
+        <alwaysOn>true</alwaysOn>
     </plugin>
   </gazebo>
@@ -25,19 +28,18 @@
   <xacro:property name="base_width" value="0.8" />
   <xacro:property name="base_height" value="1.1" />
-  <xacro:property name="base_mass" value="5" />
+  <xacro:property name="base_mass" value="30" />
   <!-- Wheel link dimensions -->
   <xacro:property name="wheel_radius" value="0.125" />
   <xacro:property name="wheel_thickness" value="0.1" />
-  <xacro:property name="wheel_mass" value="10" />
+  <xacro:property name="wheel_mass" value="2" />
   <!-- Steering link dimensions -->
-  <xacro:property name="steer_radius" value="0.08" />
+  <xacro:property name="steer_radius" value="0.05" />
   <xacro:property name="steer_thickness" value="0.02" />
   <xacro:property name="steer_mass" value="0.1" />
+  <!-- Axle positions -->
+  <xacro:property name="axle_offset" value="0.05" />
+  <xacro:property name="steer_offset" value="0.02" />
   <xacro:property name="b2f_axis_distance" value="1.1"/>
   <xacro:property name="b_axis_length" value="0.8"/>
-  <xacro:property name="base_link_to_steer_link_height" value="0.165"/>
-  <xacro:property name="general_offset" value="0.05"/>  <xacro:property name="b2f_axis_distance" value="1.1"/>
-  <xacro:property name="steer_height" value="0.9"/>
-<!--========================================================================================-->
   <!-- Base link -->
   <link name="base_link">
@@ -45,5 +47,5 @@
       <origin xyz="0 0 0" rpy="0 0 0"/>
       <geometry>
-          <mesh filename="package://hakuroukun_description/meshes/hakuroukun_base_.stl" scale="0.001 0.001 0.001" />
+          <mesh filename="package://hakuroukun_description/meshes/hakuroukun_base_link.stl" scale="0.001 0.001 0.001" />
       </geometry>
       <material name="grey"/>
@@ -52,7 +54,6 @@
       <origin xyz="0 0 0" rpy="0 0 0"/>
       <geometry>
-          <mesh filename="package://hakuroukun_description/meshes/hakuroukun_base_.stl" scale="0.001 0.001 0.001" />
+          <mesh filename="package://hakuroukun_description/meshes/hakuroukun_base_link.stl" scale="0.001 0.001 0.001" />
       </geometry>
-      <material name="grey"/>
     </collision>
     <xacro:solid_cuboid_inertial
@@ -61,6 +62,5 @@
         x="${base_length}" y="${base_width}" z="${base_height}" />
   </link>
-<!--========================================================================================-->
-  <!-- Front steer and front wheel joints -->
+  <!-- Front steer and rear wheel joints required for ackermann_steering_controller -->
   <xacro:front_steer
     name="front"
@@ -71,7 +71,7 @@
     base_length="${base_length}"
     base_width="${base_width}"
-    steer_height="${steer_height}">
+    steer_height="${wheel_radius}">
   </xacro:front_steer>
-   <xacro:front_wheel
+  <xacro:front_wheel
     name="front"
     parent="front_steer"
@@ -79,15 +79,14 @@
     wheel_thickness="${wheel_thickness}"
     wheel_mass="${wheel_mass}">
-    <origin xyz="0 0 ${-steer_height}" rpy="0 0 ${90 * deg_to_rad}"/>
+    <origin xyz="0 0 ${-wheel_radius-steer_offset}" rpy="0 0 ${90 * deg_to_rad}"/>
   </xacro:front_wheel>
-<!--========================================================================================-->
-  <!-- Rear wheels and Rear wheel left right -->
+  <!-- REAR WHEEL-->
   <xacro:rear_wheel
     name="rear"
     parent="base"
-    wheel_radius="${wheel_radius/4}"
-    wheel_thickness="${wheel_thickness/2}"
-    wheel_mass="${wheel_mass/32}">
-    <origin xyz="${-b2f_axis_distance/2} 0 0" rpy="${-90 * deg_to_rad} 0 0"/>
+    wheel_radius="${wheel_radius}"
+    wheel_thickness="${wheel_thickness}"
+    wheel_mass="${wheel_mass}">
+    <origin xyz="0 0 0" rpy="0 0 0"/>
   </xacro:rear_wheel>
   <xacro:rear_wheel_lr
@@ -97,5 +96,5 @@
     wheel_thickness="${wheel_thickness}"
     wheel_mass="${wheel_mass}">
-    <origin xyz="${-b2f_axis_distance/2} ${-b_axis_length/2} 0" rpy="0 0 0"/>
+    <origin xyz="0 ${-b_axis_length/2} 0" rpy="0 0 0"/>
   </xacro:rear_wheel_lr>
   <xacro:rear_wheel_lr
@@ -105,5 +104,5 @@
     wheel_thickness="${wheel_thickness}"
     wheel_mass="${wheel_mass}">
-    <origin xyz="${-b2f_axis_distance/2} ${+b_axis_length/2} 0" rpy="0 0 0"/>
+    <origin xyz="0 ${b_axis_length/2} 0" rpy="0 0 0"/>
   </xacro:rear_wheel_lr>
   <!-- Colour -->

File: src/hakuroukun/hakuroukun_description/urdf/robot_part/hakuroukun_wheel.xacro (robot description, xacro)
@@ -9,6 +9,6 @@
 <robot name="wheel" xmlns:xacro="http://wiki.ros.org/xacro">
   <!-- Include xacro for materials and inertials -->
-  <xacro:include filename="$(find hakuroukun_description)/urdf/robot_part/materials.xacro"/>
-  <xacro:include filename="$(find hakuroukun_description)/urdf/robot_part/inertials.xacro"/>
+  <xacro:include filename="$(find hakuroukun_description)/urdf/robot_part/hakuroukun_materials.xacro"/>
+  <xacro:include filename="$(find hakuroukun_description)/urdf/robot_part/hakuroukun_inertials.xacro"/>
   <!-- Properties -->
   <xacro:property name="steer_effort" value="10.0"/>
@@ -19,4 +19,5 @@
   <xacro:property name="b2f_axis_distance" value="1.1"/>
   <xacro:property name="b_axis_length" value="0.8"/>
+  <xacro:property name="base_link_to_steer_link_height" value="0.165"/>
   <!-- Bicycle model front steering link - FRONT REVOLUTE -->
   <xacro:macro name="front_steer"
@@ -29,5 +30,4 @@
       base_length
       base_width
-      axle_offset
       steer_height">
     <link name="${name}_steer_link">
@@ -53,8 +53,8 @@
       <parent link="${parent}_link"/>
       <child link="${name}_steer_link"/>
-      <origin xyz="${b2f_axis_distance} 0 ${steer_height}" rpy="0 0 0"/>
+      <origin xyz="${b2f_axis_distance/2} 0 ${steer_height}" rpy="0 0 0"/>
       <axis xyz="0 0 1"/>
       <limit effort="${steer_effort}"
-             lower="${-180.0 * deg_to_rad}" upper="${180.0 * deg_to_rad}"
+             lower="${-steer_limit_deg * deg_to_rad}" upper="${steer_limit_deg * deg_to_rad}"
              velocity="${steer_velocity}"/>
     </joint>
@@ -84,12 +84,12 @@
         <origin xyz="0 0 0" rpy="0 0 0"/>
         <geometry>
-          <mesh filename="package://hakuroukun_description/meshes/hakuroukun_front_wheel.stl" scale="0.001 0.001 0.001" />
-        </geometry>
-        <material name="light_grey"/>
-      </visual>
-      <collision>
-        <origin xyz="0 0 0" rpy="0 0 0"/>
-        <geometry>
-          <mesh filename="package://hakuroukun_description/meshes/hakuroukun_front_wheel.stl" scale="0.001 0.001 0.001" />
+          <mesh filename="package://hakuroukun_description/meshes/Ver2/hakuroukun_front_wheel.stl" scale="0.001 0.001 0.001" />
+        </geometry>
+        <material name="light_grey"/>
+      </visual>
+      <collision>
+        <origin xyz="0 0 0" rpy="0 0 0"/>
+        <geometry>
+          <mesh filename="package://hakuroukun_description/meshes/Ver2/hakuroukun_front_wheel.stl" scale="0.001 0.001 0.001" />
         </geometry>
       </collision>
@@ -105,14 +105,4 @@
       <axis xyz="0 1 0"/>
     </joint>
-    <!-- <transmission name="${name}_steer_joint_trans">
-      <type>transmission_interface/SimpleTransmission</type>
-      <actuator name="${name}_steer_joint_motor">
-        <mechanicalReduction>1</mechanicalReduction>
-        <hardwareInterface>hardware_interface/PositionJointInterface</hardwareInterface>
-      </actuator>
-      <joint name="${name}_wheel_joint">
-        <hardwareInterface>hardware_interface/PositionJointInterface</hardwareInterface>
-      </joint>
-    </transmission> -->
     <gazebo reference="${name}_wheel_link">
       <material>Gazebo/Grey</material>
@@ -136,12 +126,12 @@
         <origin xyz="0 0 0" rpy="0 0 0"/>
         <geometry>
-          <mesh filename="package://hakuroukun_description/meshes/hakuroukun_back_wheel.stl" scale="0.001 0.001 0.001" />
-        </geometry>
-        <material name="light_grey"/>
-      </visual>
-      <collision>
-        <origin xyz="0 0 0" rpy="0 0 0"/>
-        <geometry>
-          <mesh filename="package://hakuroukun_description/meshes/hakuroukun_back_wheel.stl" scale="0.001 0.001 0.001" />
+          <cylinder radius="${wheel_radius}" length="${wheel_thickness}"/>
+        </geometry>
+        <material name="light_grey"/>
+      </visual>
+      <collision>
+        <origin xyz="0 0 0" rpy="0 0 0"/>
+        <geometry>
+          <cylinder radius="${wheel_radius}" length="${wheel_thickness}"/>
         </geometry>
       </collision>
@@ -155,5 +145,5 @@
       <child link="${name}_wheel_link"/>
       <xacro:insert_block name="origin"/>
-      <axis xyz="0 1 0"/>
+      <axis xyz="0 0 1"/>
     </joint>
     <transmission name="${name}_wheel_joint_trans">
